File: FE_2CH/HW/v2.3/pocket_sdr_v2.3.kicad_sch (KiCad schematic)
At the start: 76 parts, among them J1 PINH_2MM_2P, J2 USB_C_Receptacle_USB2.0, J4 SMA-ANG, U1 MAX2771, U2 MAX2771, U3 CY7C68013A-56LTXCT, U4 AT24C128C, U5 LDO 3.3V 500mA SOT23-5

Commit message: JLCPCB mappings
Parts:
- AR1: LCSC (none) -> C192510
- C12, C8: LCSC (none) -> C18522294
- C14, C18, C29, C32, C33, C36, C39, C40, C41, C42: LCSC (none) -> C18504148
- C19, C20: LCSC (none) -> C18504156
- C2: LCSC (none) -> C161313
- C21: LCSC (none) -> C18498824
- C22, C24: LCSC (none) -> C730480
- C4: LCSC (none) -> C541332
- F1: LCSC (none) -> C2649924
- J2: LCSC (none) -> C3025063
- J4: LCSC (none) -> C5356059
- L1: LCSC (none) -> C341695
- L2: LCSC (none) -> C98082
- L3: LCSC (none) -> C1329831
- LED1, LED2, LED3: LCSC (none) -> C5125066
- R1, R3: LCSC (none) -> C137917
- R10, R2, R4, R6, R8: LCSC (none) -> C60489
- R11: LCSC (none) -> C106233
- R12, R13: LCSC (none) -> C4346772
- R5, R7: LCSC (none) -> C163447
- R9: LCSC (none) -> C106234
- RF_DIVIDER0: LCSC (none) -> C5136968
- TCXO0: LCSC (none) -> C7528445
- U1, U2: LCSC (none) -> C400143
- U3: LCSC (none) -> C14912
- U4: LCSC (none) -> C616767
- U5: LCSC (none) -> C3749679
Connections:
- net GND renamed CPAD_2.2MM

Commit message: Alternative JLCPCB mappings
Parts:
- C1, C15, C3, C5, C9: LCSC (none) -> C106207
- C10, C6: LCSC (none) -> C710656
- C11, C7: LCSC (none) -> C1548
- C12, C8: LCSC C18522294 -> C327009
- C13, C16, C17, C23, C25, C26, C27, C28, C30, C31, C34, C35, C37, C38, C43: LCSC (none) -> C1525
- C14, C18, C29, C32, C33, C36, C39, C40, C41, C42: LCSC C18504148 -> C1546
- C19, C20: LCSC C18504156 -> C1547
- C21: LCSC C18498824 -> C14445
- L1: LCSC C341695 -> C98081
- L3: LCSC C1329831 -> C346331
- LED1, LED2, LED3: LCSC C5125066 -> C2290
- R12, R13: LCSC C4346772 -> C25905
- XTAL0: LCSC (none) -> C255917

Commit message: Update JLCPCB mappings
Parts:
- C1, C15, C3, C5, C9: LCSC C106207 -> C126512
- C11, C7: LCSC C1548 -> C441742
- C12, C8: LCSC C327009 -> C91601
- C13, C16, C17, C23, C25, C26, C27, C28, C30, C31, C34, C35, C37, C38, C43: LCSC C1525 -> C85858
- C14, C18, C29, C32, C33, C36, C39, C40, C41, C42: LCSC C1546 -> C126492
- C19, C20: LCSC C1547 -> C85875
- C21: LCSC C14445 -> C76999
- L3: LCSC C346331 -> C1329831
Changed lines of the file:
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@@
 			)
 		)
-		(property "LCSC" "C1546"
+		(property "LCSC" "C126492"
 			(at 118.745 271.145 0)
 			(effects
@@
 			)
 		)
-		(property "LCSC" "C106207"
+		(property "LCSC" "C126512"
 			(at 86.36 90.17 0)
 			(effects
@@
 			)
 		)
-		(property "LCSC" "C1548"
+		(property "LCSC" "C441742"
 			(at 154.305 263.525 0)
 			(effects
@@
 			)
 		)
-		(property "LCSC" "C1525"
+		(property "LCSC" "C85858"
 			(at 313.055 70.485 0)
 			(effects
@@
 			)
 		)
-		(property "LCSC" "C327009"
+		(property "LCSC" "C91601"
 			(at 167.64 269.875 0)
 			(effects
@@
 			)
 		)
-		(property "LCSC" "C14445"
+		(property "LCSC" "C76999"
 			(at 343.535 131.445 0)
 			(effects
@@
 			)
 		)
-		(property "LCSC" "C1525"
+		(property "LCSC" "C85858"
 			(at 409.575 263.525 0)
 			(effects
@@
 			)
 		)
-		(property "LCSC" "C1546"
+		(property "LCSC" "C126492"
 			(at 440.055 263.525 0)
 			(effects
@@
 			)
 		)
-		(property "LCSC" "C1546"
+		(property "LCSC" "C126492"
 			(at 33.655 200.66 0)
 			(effects
@@
 			)
 		)
-		(property "LCSC" "C1546"
+		(property "LCSC" "C126492"
 			(at 42.545 271.145 0)
 			(effects
@@
 			)
 		)
-		(property "LCSC" "C1546"
+		(property "LCSC" "C126492"
 			(at 57.785 271.145 0)
 			(effects
@@
 			)
 		)
-		(property "LCSC" "C1525"
+		(property "LCSC" "C85858"
 			(at 95.885 271.145 0)
 			(effects
@@
 			)
 		)
-		(property "LCSC" "C1546"
+		(property "LCSC" "C126492"
 			(at 50.165 271.145 0)
 			(effects
@@
 			)
 		)
-		(property "LCSC" "C1525"
+		(property "LCSC" "C85858"
 			(at 13.97 97.79 0)
 			(effects
@@
 			)
 		)
-		(property "LCSC" "C1547"
+		(property "LCSC" "C85875"
 			(at 310.515 149.86 0)
 			(effects
@@
 			)
 		)
-		(property "LCSC" "C1525"
+		(property "LCSC" "C85858"
 			(at 65.405 271.145 0)
 			(effects
@@
 			)
 		)
-		(property "LCSC" "C106207"
+		(property "LCSC" "C126512"
 			(at 30.48 161.29 0)
 			(effects
@@
 			)
 		)
-		(property "LCSC" "C1546"
+		(property "LCSC" "C126492"
 			(at 80.645 271.145 0)
 			(effects
@@
 			)
 		)
-		(property "LCSC" "C1525"
+		(property "LCSC" "C85858"
 			(at 111.125 271.145 0)
 			(effects
@@
 			)
 		)
-		(property "LCSC" "C1525"
+		(property "LCSC" "C85858"
 			(at 41.275 200.66 0)
 			(effects
@@
 			)
 		)
-		(property "LCSC" "C1525"
+		(property "LCSC" "C85858"
 			(at 12.065 271.145 0)
 			(effects
@@
 			)
 		)
-		(property "LCSC" "C1525"
+		(property "LCSC" "C85858"
 			(at 88.265 271.145 0)
 			(effects
@@
 			)
 		)
-		(property "LCSC" "C1547"
+		(property "LCSC" "C85875"
 			(at 310.515 170.18 0)
 			(effects
@@
 			)
 		)
-		(property "LCSC" "C1525"
+		(property "LCSC" "C85858"
 			(at 417.195 263.525 0)
 			(effects
@@
 			)
 		)
-		(property "LCSC" "C1525"
+		(property "LCSC" "C85858"
 			(at 73.025 271.145 0)
 			(effects
@@
 			)
 		)
-		(property "LCSC" "C106207"
+		(property "LCSC" "C126512"
 			(at 125.73 102.87 0)
 			(effects
@@
 			)
 		)
-		(property "LCSC" "C1546"
+		(property "LCSC" "C126492"
 			(at 27.305 271.145 0)
 			(effects
@@
 			)
 		)
-		(property "LCSC" "C346331"
+		(property "LCSC" "C1329831"
 			(at 99.314 232.918 0)
 			(effects
@@
 			)
 		)
-		(property "LCSC" "C1525"
+		(property "LCSC" "C85858"
 			(at 366.395 263.525 0)
 			(effects
@@
 			)
 		)
-		(property "LCSC" "C327009"
+		(property "LCSC" "C91601"
 			(at 167.005 153.035 0)
 			(effects
@@
 			)
 		)
-		(property "LCSC" "C1548"
+		(property "LCSC" "C441742"
 			(at 154.305 146.685 0)
 			(effects
@@
 			)
 		)
-		(property "LCSC" "C1525"
+		(property "LCSC" "C85858"
 			(at 424.815 263.525 0)
 			(effects
@@
 			)
 		)
-		(property "LCSC" "C1525"
+		(property "LCSC" "C85858"
 			(at 19.685 271.145 0)
 			(effects
@@
 			)
 		)
-		(property "LCSC" "C1525"
+		(property "LCSC" "C85858"
 			(at 34.925 271.145 0)
 			(effects
@@
 			)
 		)
-		(property "LCSC" "C106207"
+		(property "LCSC" "C126512"
 			(at 86.36 232.41 0)
 			(effects
@@
 			)
 		)
-		(property "LCSC" "C1546"
+		(property "LCSC" "C126492"
 			(at 432.435 263.525 0)
 			(effects
@@
 			)
 		)
-		(property "LCSC" "C106207"
+		(property "LCSC" "C126512"
 			(at 118.11 219.71 0)
 			(effects
@@
 			)
 		)
-		(property "LCSC" "C1546"
+		(property "LCSC" "C126492"
 			(at 103.505 271.145 0)
 			(effects

Commit message: Fix USB-C footprint assignment
Parts:
- C1, C15, C3, C5, C9: LCSC C126512 -> C106207
- C11, C7: LCSC C441742 -> C1548
- C12, C8: LCSC C91601 -> C327009
- C13, C16, C17, C23, C25, C26, C27, C28, C30, C31, C34, C35, C37, C38, C43: LCSC C85858 -> C1525
- C14, C18, C29, C32, C33, C36, C39, C40, C41, C42: LCSC C126492 -> C1546
- C19, C20: LCSC C85875 -> C1547
- C21: LCSC C76999 -> C14445
- J2: footprint (none) -> Connector_USB:USB_C_Receptacle_GCT_USB4105-xx-A_16P_TopMnt_Horizontal
- L3: LCSC C1329831 -> C346331
Changed lines of the file:
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@@
 			)
 		)
-		(property "LCSC" "C126492"
+		(property "LCSC" "C1546"
 			(at 118.745 271.145 0)
 			(effects
@@
 			)
 		)
-		(property "LCSC" "C126512"
+		(property "LCSC" "C106207"
 			(at 86.36 90.17 0)
 			(effects
@@
 			)
 		)
-		(property "LCSC" "C441742"
+		(property "LCSC" "C1548"
 			(at 154.305 263.525 0)
 			(effects
@@
 			)
 		)
-		(property "LCSC" "C85858"
+		(property "LCSC" "C1525"
 			(at 313.055 70.485 0)
 			(effects
@@
 			)
 		)
-		(property "LCSC" "C91601"
+		(property "LCSC" "C327009"
 			(at 167.64 269.875 0)
 			(effects
@@
 			)
 		)
-		(property "LCSC" "C76999"
+		(property "LCSC" "C14445"
 			(at 343.535 131.445 0)
 			(effects
@@
 			)
 		)
-		(property "LCSC" "C85858"
+		(property "LCSC" "C1525"
 			(at 409.575 263.525 0)
 			(effects
@@
 			)
 		)
-		(property "LCSC" "C126492"
+		(property "LCSC" "C1546"
 			(at 440.055 263.525 0)
 			(effects
@@
 			)
 		)
-		(property "LCSC" "C126492"
+		(property "LCSC" "C1546"
 			(at 33.655 200.66 0)
 			(effects
@@
 			)
 		)
-		(property "LCSC" "C126492"
+		(property "LCSC" "C1546"
 			(at 42.545 271.145 0)
 			(effects
@@
 			)
 		)
-		(property "LCSC" "C126492"
+		(property "LCSC" "C1546"
 			(at 57.785 271.145 0)
 			(effects
@@
 			)
 		)
-		(property "LCSC" "C85858"
+		(property "LCSC" "C1525"
 			(at 95.885 271.145 0)
 			(effects
@@
 			)
 		)
-		(property "LCSC" "C126492"
+		(property "LCSC" "C1546"
 			(at 50.165 271.145 0)
 			(effects
@@
 			)
 		)
-		(property "LCSC" "C85858"
+		(property "LCSC" "C1525"
 			(at 13.97 97.79 0)
 			(effects
@@
 			)
 		)
-		(property "LCSC" "C85875"
+		(property "LCSC" "C1547"
 			(at 310.515 149.86 0)
 			(effects
@@
 			)
 		)
-		(property "LCSC" "C85858"
+		(property "LCSC" "C1525"
 			(at 65.405 271.145 0)
 			(effects
@@
 			)
 		)
-		(property "LCSC" "C126512"
+		(property "LCSC" "C106207"
 			(at 30.48 161.29 0)
 			(effects
@@
 			)
 		)
-		(property "LCSC" "C126492"
+		(property "LCSC" "C1546"
 			(at 80.645 271.145 0)
 			(effects
@@
 			)
 		)
-		(property "LCSC" "C85858"
+		(property "LCSC" "C1525"
 			(at 111.125 271.145 0)
 			(effects
@@
 			)
 		)
-		(property "LCSC" "C85858"
+		(property "LCSC" "C1525"
 			(at 41.275 200.66 0)
 			(effects
@@
 			)
 		)
-		(property "LCSC" "C85858"
+		(property "LCSC" "C1525"
 			(at 12.065 271.145 0)
 			(effects
@@
 			)
 		)
-		(property "LCSC" "C85858"
+		(property "LCSC" "C1525"
 			(at 88.265 271.145 0)
 			(effects
@@
 			)
 		)
-		(property "Footprint" ""
+		(property "Footprint" "Connector_USB:USB_C_Receptacle_GCT_USB4105-xx-A_16P_TopMnt_Horizontal"
 			(at 306.07 255.27 0)
 			(effects
@@
 			)
 		)
-		(property "LCSC" "C85875"
+		(property "LCSC" "C1547"
 			(at 310.515 170.18 0)
 			(effects
@@
 			)
 		)
-		(property "LCSC" "C85858"
+		(property "LCSC" "C1525"
 			(at 417.195 263.525 0)
 			(effects
@@
 			)
 		)
-		(property "LCSC" "C85858"
+		(property "LCSC" "C1525"
 			(at 73.025 271.145 0)
 			(effects
@@
 			)
 		)
-		(property "LCSC" "C126512"
+		(property "LCSC" "C106207"
 			(at 125.73 102.87 0)
 			(effects
@@
 			)
 		)
-		(property "LCSC" "C126492"
+		(property "LCSC" "C1546"
 			(at 27.305 271.145 0)
 			(effects
@@
 			)
 		)
-		(property "LCSC" "C1329831"
+		(property "LCSC" "C346331"
 			(at 99.314 232.918 0)
 			(effects
@@
 			)
 		)
-		(property "LCSC" "C85858"
+		(property "LCSC" "C1525"
 			(at 366.395 263.525 0)
 			(effects
@@
 			)
 		)
-		(property "LCSC" "C91601"
+		(property "LCSC" "C327009"
 			(at 167.005 153.035 0)
 			(effects
@@
 			)
 		)
-		(property "LCSC" "C441742"
+		(property "LCSC" "C1548"
 			(at 154.305 146.685 0)
 			(effects
@@
 			)
 		)
-		(property "LCSC" "C85858"
+		(property "LCSC" "C1525"
 			(at 424.815 263.525 0)
 			(effects
@@
 			)
 		)
-		(property "LCSC" "C85858"
+		(property "LCSC" "C1525"
 			(at 19.685 271.145 0)
 			(effects
@@
 			)
 		)
-		(property "LCSC" "C85858"
+		(property "LCSC" "C1525"
 			(at 34.925 271.145 0)
 			(effects
@@
 			)
 		)
-		(property "LCSC" "C126512"
+		(property "LCSC" "C106207"
 			(at 86.36 232.41 0)
 			(effects
@@
 			)
 		)
-		(property "LCSC" "C126492"
+		(property "LCSC" "C1546"
 			(at 432.435 263.525 0)
 			(effects
@@
 			)
 		)
-		(property "LCSC" "C126512"
+		(property "LCSC" "C106207"
 			(at 118.11 219.71 0)
 			(effects
@@
 			)
 		)
-		(property "LCSC" "C126492"
+		(property "LCSC" "C1546"
 			(at 103.505 271.145 0)
 			(effects

Commit message: Put back bias tee and U.FL connector
Parts:
- removed C15: 470pF, pocket_sdr_v2.3:C1005, symbol pocket_sdr_v2.3-eagle-import:C1005
- removed C43: 0.1uF, pocket_sdr_v2.3:C1005, symbol pocket_sdr_v2.3-eagle-import:C1005
- removed F1: 12V 8 Ohm, Trip 250mA, pocket_sdr_v2.3:C1608, symbol pocket_sdr_v2.3-eagle-import:POLYSW1608
- removed J4: SMA-ANG, pocket_sdr_v2.3:SMA-ANG, symbol pocket_sdr_v2.3-eagle-import:SMA-ANG
- removed L2: 68nH, pocket_sdr_v2.3:C1608, symbol pocket_sdr_v2.3-eagle-import:L1608
- added IC1: TCBT-2R5G+, LIB_TCBT-2R5G+:TCBT2R5G, symbol TCBT-2R5G+:TCBT-2R5G+
- added J3: ANT POWER, Connector_PinHeader_2.00mm:PinHeader_1x02_P2.00mm_Vertical, symbol Connector_Generic:Conn_01x02
- added J4: U.FL-R-SMT-1_80_, LIB_U.FL-R-SMT-1_80_:UFLRSMT180, symbol U_FL-R-SMT-1_80_:U.FL-R-SMT-1_80_
- C14: value 100pF -> 0.01uF
Connections:
- net 5V: now also J3.1 (Pin_1)
- net CPAD_2.2MM: now also IC1.2 (ISOLATE), J4.2 (GND_1), J4.3 (GND_2)
- net at RF_DIVIDER0.2 (INPUT): now also IC1.4 (RF)
- net at C14.2: now also IC1.1 (DC), J3.2 (Pin_2)
- new net: IC1.3 (RF&DC), J4.1 (SIG)
Other:
- moved on the sheet: AR1, C1, C10, C11, C12, C13, C14, C16, C17, C18, C19, C2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
